Commit message: Affix all joints except for the elbow

File: arm_1dof/demo_human_col/skeleton.urdf (robot description, URDF)
Before this commit: robot skeleton, 10 links, 9 joints
Joints:
- joint skeleton__distal_joint: type revolute -> fixed
- joint skeleton__middle_joint: type revolute -> fixed
- joint skeleton__proximal_joint: type revolute -> fixed
- joint skeleton__shoulder_joint: type revolute -> fixed

Commit message: Realistic upper and forearm weights

File: arm_1dof/demo_human_col/skeleton.urdf (robot description, URDF)
Before this commit: robot skeleton, 10 links, 9 joints
Links:
- link skeleton__distal: mass 0.19999998807907104 -> 0.001
- link skeleton__forearm: mass 0.19999998807907104 -> 1.89
- link skeleton__hand: mass 0.19999998807907104 -> 0.001
- link skeleton__middle: mass 0.19999998807907104 -> 0.001
- link skeleton__proximal: mass 0.19999998807907104 -> 0.001
- link skeleton__skeleton: mass 0.20000000298023224 -> 1.0
- link skeleton__thumb_1: mass 0.19999998807907104 -> 0.001
- link skeleton__thumb_2: mass 0.19999998807907104 -> 0.001
- link skeleton__thumb_3: mass 0.19999998807907104 -> 0.001
- link skeleton__upper_arm: mass 0.19999998807907104 -> 2.4375
